File: pcb/Seven_segment_Eight_ShiftRegisters/Seven_segment_Eight_ShiftRegisters.kicad_pcb (KiCad board)
At the start: 2 copper layers, 18 parts, among them Q1 TIP120, Q2 TIP120, Q3 TIP120, Q4 TIP120, Q5 TIP120

Commit message: sync
Parts:
- added J1: B5B-XH-A_LF__SN_, Connector_PinHeader_2.00mm:PinHeader_1x05_P2.00mm_Vertical, F.Cu at (59.8, 151.3)
- added J2: B3B-PH-K-S_LF__SN_, Connector_PinHeader_2.00mm:PinHeader_1x03_P2.00mm_Vertical, F.Cu at (67.7, 180.5)
- added U1: 5161AS, HariLib:5161AS, F.Cu at (166.1, 36.3)
- added U10: 5161AS, HariLib:5161AS, F.Cu at (85.7, 120.4)
- added U11: 5161AS, HariLib:5161AS, F.Cu at (83.3, 139.7)
- added U12: 74HC595, Package_SO:SOIC-16_3.9x9.9mm_P1.27mm, B.Cu at (91.7, 173.5)
- added U13: 5161AS, HariLib:5161AS, F.Cu at (138.2, 15.9)
- added U14: 5161AS, HariLib:5161AS, F.Cu at (180.1, 36.3)
- added U15: 5161AS, HariLib:5161AS, F.Cu at (152.2, 56.6)
- added U16: 5161AS, HariLib:5161AS, F.Cu at (138.2, 77.0)
- added U17: 5161AS, HariLib:5161AS, F.Cu at (194.0, 36.3)
- added U18: 74HC595, Package_SO:SOIC-16_3.9x9.9mm_P1.27mm, F.Cu at (267.2, 61.6)
- added U19: 5161AS, HariLib:5161AS, F.Cu at (152.2, 77.0)
- added U2: 5161AS, HariLib:5161AS, F.Cu at (124.2, 56.6)
- added U20: 5161AS, HariLib:5161AS, F.Cu at (166.1, 56.6)
- added U21: 5161AS, HariLib:5161AS, F.Cu at (207.9, 15.9)
- added U22: 5161AS, HariLib:5161AS, F.Cu at (180.1, 56.6)
- added U23: 5161AS, HariLib:5161AS, F.Cu at (194.0, 56.6)
- added U24: 74HC595, Package_SO:SOIC-16_3.9x9.9mm_P1.27mm, F.Cu at (247.8, 82.0)
- added U25: 5161AS, HariLib:5161AS, F.Cu at (235.8, 36.3)
- added U26: 5161AS, HariLib:5161AS, F.Cu at (194.0, 15.9)
- added U27: 5161AS, HariLib:5161AS, F.Cu at (207.9, 77.0)
- added U28: 5161AS, HariLib:5161AS, F.Cu at (207.9, 56.6)
- added U29: 5161AS, HariLib:5161AS, F.Cu at (207.9, 36.3)
- added U3: 5161AS, HariLib:5161AS, F.Cu at (76.0, 101.3)
- added U30: 74HC595, Package_SO:SOIC-16_3.9x9.9mm_P1.27mm, F.Cu at (239.3, 93.4)
- added U31: 5161AS, HariLib:5161AS, F.Cu at (166.1, 77.0)
- added U32: 5161AS, HariLib:5161AS, F.Cu at (180.1, 77.0)
- added U33: 5161AS, HariLib:5161AS, F.Cu at (235.8, 15.9)
- added U34: 5161AS, HariLib:5161AS, F.Cu at (194.0, 77.0)
- added U35: 5161AS, HariLib:5161AS, F.Cu at (249.8, 15.9)
- added U36: 74HC595, Package_SO:SOIC-16_3.9x9.9mm_P1.27mm, F.Cu at (247.8, 93.4)
- added U37: 5161AS, HariLib:5161AS, F.Cu at (235.8, 56.6)
- added U38: 5161AS, HariLib:5161AS, F.Cu at (221.9, 15.9)
- added U39: 5161AS, HariLib:5161AS, F.Cu at (249.8, 36.3)
- added U4: 5161AS, HariLib:5161AS, F.Cu at (73.2, 120.5)
- added U40: 5161AS, HariLib:5161AS, F.Cu at (221.9, 56.6)
- added U41: 5161AS, HariLib:5161AS, F.Cu at (263.8, 15.9)
- added U42: 74HC595, Package_SO:SOIC-16_3.9x9.9mm_P1.27mm, F.Cu at (267.2, 73.1)
- added U43: 5161AS, HariLib:5161AS, F.Cu at (249.8, 56.6)
- added U44: 5161AS, HariLib:5161AS, F.Cu at (263.8, 36.3)
- added U45: 5161AS, HariLib:5161AS, F.Cu at (221.9, 77.0)
- added U46: 5161AS, HariLib:5161AS, F.Cu at (221.9, 36.3)
- added U47: 5161AS, HariLib:5161AS, F.Cu at (124.2, 36.3)
- added U48: 74HC595, Package_SO:SOIC-16_3.9x9.9mm_P1.27mm, F.Cu at (256.2, 82.0)
- added U5: 5161AS, HariLib:5161AS, F.Cu at (70.4, 139.7)
- added U6: 74HC595, Package_SO:SOIC-16_3.9x9.9mm_P1.27mm, B.Cu at (77.0, 173.6)
- added U7: 5161AS, HariLib:5161AS, F.Cu at (152.2, 36.3)
- added U8: 5161AS, HariLib:5161AS, F.Cu at (138.2, 56.6)
- added U9: 5161AS, HariLib:5161AS, F.Cu at (166.1, 15.9)
- RN1, RN2, RN3, RN4, RN5, RN6, RN7, RN8: footprint HariLib:EXB-2HV221JV -> EXB-2HV221JV:EXB-2HV221JV
- moved RN1 152.9 mm to (80.8, 162.4), turned to 90 degrees
- moved RN2 152.7 mm to (92.6, 162.7), turned to 90 degrees
- moved Q5 117.3 mm to (67.0, 151.3), turned to 90 degrees
- moved R5 113.5 mm to (63.4, 151.3), turned to 180 degrees
- moved RN5 39.8 mm to (26.2, 76.8)
- moved RN6 39.8 mm to (33.6, 76.8)
- moved Q1 39.8 mm to (58.1, 57.3)
- moved Q2 39.8 mm to (58.1, 63.3)
- moved Q3 39.8 mm to (69.7, 57.3)
- moved Q4 39.8 mm to (58.1, 69.2)
- moved R1 39.8 mm to (39.0, 72.8)
- moved R2 39.8 mm to (39.0, 75.3)
- moved R3 39.8 mm to (43.3, 72.8)
- moved R4 39.8 mm to (43.3, 75.3)
- moved RN3 39.8 mm to (26.2, 66.3)
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Connections:
- Q1 pad 2: (no net) -> Net-(Q1-Pad2)
- Q2 pad 2: (no net) -> Net-(Q2-Pad2)
- Q3 pad 2: (no net) -> Net-(Q3-Pad2)
- Q4 pad 2: (no net) -> Net-(Q4-Pad2)
- Q5 pad 2: (no net) -> Net-(Q5-Pad2)
- R1 pad 2: (no net) -> Net-(J1-Pad4)
- R2 pad 2: (no net) -> Net-(J1-Pad2)
- R3 pad 2: (no net) -> Net-(J1-Pad5)
- R4 pad 2: (no net) -> Net-(J1-Pad3)
- R5 pad 2: (no net) -> Net-(J1-Pad1)
- RN1 pad 1: (no net) -> Net-(RN1-Pad1)
- RN1 pad 10: (no net) -> Net-(RN1-Pad10)
- RN1 pad 11: (no net) -> Net-(RN1-Pad11)
- RN1 pad 12: (no net) -> Net-(RN1-Pad12)
- RN1 pad 13: (no net) -> Net-(RN1-Pad13)
- RN1 pad 14: (no net) -> Net-(RN1-Pad14)
- RN1 pad 15: (no net) -> Net-(RN1-Pad15)
- RN1 pad 16: (no net) -> Net-(RN1-Pad16)
- RN1 pad 2: (no net) -> Net-(RN1-Pad2)
- RN1 pad 3: (no net) -> Net-(RN1-Pad3)
- RN1 pad 4: (no net) -> Net-(RN1-Pad4)
- RN1 pad 5: (no net) -> Net-(RN1-Pad5)
- RN1 pad 6: (no net) -> Net-(RN1-Pad6)
- RN1 pad 7: (no net) -> Net-(RN1-Pad7)
- RN1 pad 8: (no net) -> Net-(RN1-Pad8)
- RN1 pad 9: (no net) -> Net-(RN1-Pad9)
- RN2 pad 1: (no net) -> Net-(RN2-Pad1)
- RN2 pad 10: (no net) -> Net-(RN2-Pad10)
- RN2 pad 11: (no net) -> Net-(RN2-Pad11)
- RN2 pad 12: (no net) -> Net-(RN2-Pad12)
- RN2 pad 13: (no net) -> Net-(RN2-Pad13)
- RN2 pad 14: (no net) -> Net-(RN2-Pad14)
- RN2 pad 15: (no net) -> Net-(RN2-Pad15)
- RN2 pad 16: (no net) -> Net-(RN2-Pad16)
- RN2 pad 2: (no net) -> Net-(RN2-Pad2)
- RN2 pad 3: (no net) -> Net-(RN2-Pad3)
- RN2 pad 4: (no net) -> Net-(RN2-Pad4)
- RN2 pad 5: (no net) -> Net-(RN2-Pad5)
- RN2 pad 6: (no net) -> Net-(RN2-Pad6)
- RN2 pad 7: (no net) -> Net-(RN2-Pad7)
- RN2 pad 8: (no net) -> Net-(RN2-Pad8)
- RN2 pad 9: (no net) -> Net-(RN2-Pad9)
- RN3 pad 1: (no net) -> Net-(RN3-Pad1)
- RN3 pad 10: (no net) -> Net-(RN3-Pad10)
- RN3 pad 11: (no net) -> Net-(RN3-Pad11)
- RN3 pad 12: (no net) -> Net-(RN3-Pad12)
- RN3 pad 13: (no net) -> Net-(RN3-Pad13)
- RN3 pad 14: (no net) -> Net-(RN3-Pad14)
- RN3 pad 15: (no net) -> Net-(RN3-Pad15)
- RN3 pad 16: (no net) -> Net-(RN3-Pad16)
- RN3 pad 2: (no net) -> Net-(RN3-Pad2)
- RN3 pad 3: (no net) -> Net-(RN3-Pad3)
- RN3 pad 4: (no net) -> Net-(RN3-Pad4)
- RN3 pad 5: (no net) -> Net-(RN3-Pad5)
- RN3 pad 6: (no net) -> Net-(RN3-Pad6)
- RN3 pad 7: (no net) -> Net-(RN3-Pad7)
- RN3 pad 8: (no net) -> Net-(RN3-Pad8)
- RN3 pad 9: (no net) -> Net-(RN3-Pad9)
- RN4 pad 1: (no net) -> Net-(RN4-Pad1)
- RN4 pad 10: (no net) -> Net-(RN4-Pad10)
- RN4 pad 11: (no net) -> Net-(RN4-Pad11)
- RN4 pad 12: (no net) -> Net-(RN4-Pad12)
- RN4 pad 13: (no net) -> Net-(RN4-Pad13)
- RN4 pad 14: (no net) -> Net-(RN4-Pad14)
- RN4 pad 15: (no net) -> Net-(RN4-Pad15)
- RN4 pad 16: (no net) -> Net-(RN4-Pad16)
- RN4 pad 2: (no net) -> Net-(RN4-Pad2)
- RN4 pad 3: (no net) -> Net-(RN4-Pad3)
- RN4 pad 4: (no net) -> Net-(RN4-Pad4)
- RN4 pad 5: (no net) -> Net-(RN4-Pad5)
- RN4 pad 6: (no net) -> Net-(RN4-Pad6)
- RN4 pad 7: (no net) -> Net-(RN4-Pad7)
- RN4 pad 8: (no net) -> Net-(RN4-Pad8)
- RN4 pad 9: (no net) -> Net-(RN4-Pad9)
- RN5 pad 1: (no net) -> Net-(RN5-Pad1)
- RN5 pad 10: (no net) -> Net-(RN5-Pad10)
- RN5 pad 11: (no net) -> Net-(RN5-Pad11)
- RN5 pad 12: (no net) -> Net-(RN5-Pad12)
- RN5 pad 13: (no net) -> Net-(RN5-Pad13)
- RN5 pad 14: (no net) -> Net-(RN5-Pad14)
- RN5 pad 15: (no net) -> Net-(RN5-Pad15)
- RN5 pad 16: (no net) -> Net-(RN5-Pad16)
- RN5 pad 2: (no net) -> Net-(RN5-Pad2)
- RN5 pad 3: (no net) -> Net-(RN5-Pad3)
- RN5 pad 4: (no net) -> Net-(RN5-Pad4)
- RN5 pad 5: (no net) -> Net-(RN5-Pad5)
- RN5 pad 6: (no net) -> Net-(RN5-Pad6)
- RN5 pad 7: (no net) -> Net-(RN5-Pad7)
- RN5 pad 8: (no net) -> Net-(RN5-Pad8)
- RN5 pad 9: (no net) -> Net-(RN5-Pad9)
- RN6 pad 1: (no net) -> Net-(RN6-Pad1)
- RN6 pad 10: (no net) -> Net-(RN6-Pad10)
- RN6 pad 11: (no net) -> Net-(RN6-Pad11)
- RN6 pad 12: (no net) -> Net-(RN6-Pad12)
- RN6 pad 13: (no net) -> Net-(RN6-Pad13)
- RN6 pad 14: (no net) -> Net-(RN6-Pad14)
- RN6 pad 15: (no net) -> Net-(RN6-Pad15)
- RN6 pad 16: (no net) -> Net-(RN6-Pad16)
- RN6 pad 2: (no net) -> Net-(RN6-Pad2)
- RN6 pad 3: (no net) -> Net-(RN6-Pad3)
- RN6 pad 4: (no net) -> Net-(RN6-Pad4)
- RN6 pad 5: (no net) -> Net-(RN6-Pad5)
- RN6 pad 6: (no net) -> Net-(RN6-Pad6)
- RN6 pad 7: (no net) -> Net-(RN6-Pad7)
- RN6 pad 8: (no net) -> Net-(RN6-Pad8)
- RN6 pad 9: (no net) -> Net-(RN6-Pad9)
- RN7 pad 1: (no net) -> Net-(RN7-Pad1)
- RN7 pad 10: (no net) -> Net-(RN7-Pad10)
- RN7 pad 11: (no net) -> Net-(RN7-Pad11)
- RN7 pad 12: (no net) -> Net-(RN7-Pad12)
- RN7 pad 13: (no net) -> Net-(RN7-Pad13)
- RN7 pad 14: (no net) -> Net-(RN7-Pad14)
- RN7 pad 15: (no net) -> Net-(RN7-Pad15)
- RN7 pad 16: (no net) -> Net-(RN7-Pad16)
- RN7 pad 2: (no net) -> Net-(RN7-Pad2)
- RN7 pad 3: (no net) -> Net-(RN7-Pad3)
- RN7 pad 4: (no net) -> Net-(RN7-Pad4)
- RN7 pad 5: (no net) -> Net-(RN7-Pad5)
- RN7 pad 6: (no net) -> Net-(RN7-Pad6)
- RN7 pad 7: (no net) -> Net-(RN7-Pad7)
- RN7 pad 8: (no net) -> Net-(RN7-Pad8)
- RN7 pad 9: (no net) -> Net-(RN7-Pad9)
- RN8 pad 1: (no net) -> Net-(RN8-Pad1)
- RN8 pad 10: (no net) -> Net-(RN8-Pad10)
- RN8 pad 11: (no net) -> Net-(RN8-Pad11)
- RN8 pad 12: (no net) -> Net-(RN8-Pad12)
- RN8 pad 13: (no net) -> Net-(RN8-Pad13)
- RN8 pad 14: (no net) -> Net-(RN8-Pad14)
- RN8 pad 15: (no net) -> Net-(RN8-Pad15)
- RN8 pad 16: (no net) -> Net-(RN8-Pad16)
- RN8 pad 2: (no net) -> Net-(RN8-Pad2)
- RN8 pad 3: (no net) -> Net-(RN8-Pad3)
- RN8 pad 4: (no net) -> Net-(RN8-Pad4)
- RN8 pad 5: (no net) -> Net-(RN8-Pad5)
- RN8 pad 6: (no net) -> Net-(RN8-Pad6)
- RN8 pad 7: (no net) -> Net-(RN8-Pad7)
- RN8 pad 8: (no net) -> Net-(RN8-Pad8)
- RN8 pad 9: (no net) -> Net-(RN8-Pad9)
Routing:
- net Net-(J2-Pad3): track 0.00 -> 55.8 mm, vias 0 -> 2
- net Net-(RN1-Pad12): track 0.00 -> 53.6 mm
- net Net-(Q5-Pad2): track 0.00 -> 53.1 mm, vias 0 -> 2
- net Net-(RN1-Pad10): track 0.00 -> 52.9 mm
- net Net-(RN1-Pad13): track 0.00 -> 50.8 mm, vias 0 -> 2
- net Net-(RN1-Pad11): track 0.00 -> 47.5 mm, vias 0 -> 2
- net Net-(J2-Pad2): track 0.00 -> 46.8 mm, vias 0 -> 2
- net Net-(RN1-Pad9): track 0.00 -> 45.6 mm
- net Net-(RN1-Pad15): track 0.00 -> 41.9 mm, vias 0 -> 2
- net Net-(RN1-Pad16): track 0.00 -> 41.0 mm
- net +5V: track 0.00 -> 32.0 mm
- net Net-(RN2-Pad12): track 0.00 -> 31.8 mm
- net Net-(RN2-Pad13): track 0.00 -> 29.8 mm, vias 0 -> 2
- net Net-(RN2-Pad10): track 0.00 -> 29.7 mm
- net Net-(RN2-Pad11): track 0.00 -> 26.6 mm, vias 0 -> 2
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- added copper zone on B.Cu, net GND

Commit message: About to duplicate 3d models
Routing:
- net Net-(J2-Pad3): track 55.8 -> 41.7 mm
- net Net-(J2-Pad2): track 46.8 -> 38.9 mm
