File: pcb/Seven_segment_Eight_ShiftRegisters/Seven_segment_Eight_ShiftRegisters.kicad_pcb (KiCad board)
At the start: 2 copper layers, 68 parts, among them J1 B5B-XH-A_LF__SN_, J2 B3B-PH-K-S_LF__SN_, Q1 TIP120, Q2 TIP120, Q3 TIP120, Q4 TIP120, Q5 TIP120, U1 5161AS, U10 5161AS, U11 5161AS, U12 74HC595, U13 5161AS, U14 5161AS, U15 5161AS, U16 5161AS, U17 5161AS, U18 74HC595, U19 5161AS, U2 5161AS, U20 5161AS, U21 5161AS, U22 5161AS, U23 5161AS, U24 74HC595, U25 5161AS, U26 5161AS, U27 5161AS, U28 5161AS, U29 5161AS, U3 5161AS, U30 74HC595, U31 5161AS, U32 5161AS, U33 5161AS, U34 5161AS, U35 5161AS, U36 74HC595, U37 5161AS, U38 5161AS, U39 5161AS, U4 5161AS, U40 5161AS, U41 5161AS, U42 74HC595, U43 5161AS, U44 5161AS, U45 5161AS, U46 5161AS, U47 5161AS, U48 74HC595, U5 5161AS, U6 74HC595, U7 5161AS, U8 5161AS, U9 5161AS

Commit message: Redid pcb from scratch. Got ratsnest cleaned.
Parts:
- removed U10, U11, U13, U14, U15, U16, U17, U19, U20, U21, U22, U23, U25, U26, U27, U28, U29, U31, U32, U33, U34, U35, U37, U38, U39, U40, U41, U43, U44, U45, U46, U47, U9: 5161AS, HariLib:5161AS
- removed U12, U18, U24, U30, U36, U42, U48: 74HC595, Package_SO:SOIC-16_3.9x9.9mm_P1.27mm
- added DS1: 5161AS, HariLib:5161AS, F.Cu at (127.0, 50.8)
- added DS10: 5161AS, HariLib:5161AS, F.Cu at (139.7, 71.1)
- added DS11: 5161AS, HariLib:5161AS, F.Cu at (152.4, 71.1)
- added DS12: 5161AS, HariLib:5161AS, F.Cu at (165.1, 71.1)
- added DS13: 5161AS, HariLib:5161AS, F.Cu at (177.8, 71.1)
- added DS14: 5161AS, HariLib:5161AS, F.Cu at (190.5, 71.1)
- added DS15: 5161AS, HariLib:5161AS, F.Cu at (203.2, 71.1)
- added DS16: 5161AS, HariLib:5161AS, F.Cu at (215.9, 71.1)
- added DS17: 5161AS, HariLib:5161AS, F.Cu at (127.0, 94.0)
- added DS18: 5161AS, HariLib:5161AS, F.Cu at (139.7, 94.0)
- added DS19: 5161AS, HariLib:5161AS, F.Cu at (152.4, 94.0)
- added DS2: 5161AS, HariLib:5161AS, F.Cu at (139.7, 50.8)
- added DS20: 5161AS, HariLib:5161AS, F.Cu at (165.1, 94.0)
- added DS21: 5161AS, HariLib:5161AS, F.Cu at (177.8, 94.0)
- added DS22: 5161AS, HariLib:5161AS, F.Cu at (190.5, 94.0)
- added DS23: 5161AS, HariLib:5161AS, F.Cu at (203.2, 94.0)
- added DS24: 5161AS, HariLib:5161AS, F.Cu at (215.9, 94.0)
- added DS25: 5161AS, HariLib:5161AS, F.Cu at (127.0, 114.3)
- added DS26: 5161AS, HariLib:5161AS, F.Cu at (139.7, 114.3)
- added DS27: 5161AS, HariLib:5161AS, F.Cu at (152.4, 114.3)
- added DS28: 5161AS, HariLib:5161AS, F.Cu at (165.1, 114.3)
- added DS29: 5161AS, HariLib:5161AS, F.Cu at (177.8, 114.3)
- added DS3: 5161AS, HariLib:5161AS, F.Cu at (152.4, 50.8)
- added DS30: 5161AS, HariLib:5161AS, F.Cu at (190.5, 114.3)
- added DS31: 5161AS, HariLib:5161AS, F.Cu at (203.2, 114.3)
- added DS32: 5161AS, HariLib:5161AS, F.Cu at (215.9, 114.3)
- added DS33: 5161AS, HariLib:5161AS, F.Cu at (127.0, 134.6)
- added DS34: 5161AS, HariLib:5161AS, F.Cu at (139.7, 134.6)
- added DS35: 5161AS, HariLib:5161AS, F.Cu at (152.4, 134.6)
- added DS36: 5161AS, HariLib:5161AS, F.Cu at (165.1, 134.6)
- added DS37: 5161AS, HariLib:5161AS, F.Cu at (177.8, 134.6)
- added DS38: 5161AS, HariLib:5161AS, F.Cu at (190.5, 134.6)
- added DS39: 5161AS, HariLib:5161AS, F.Cu at (203.2, 134.6)
- added DS4: 5161AS, HariLib:5161AS, F.Cu at (165.1, 50.8)
- added DS40: 5161AS, HariLib:5161AS, F.Cu at (215.9, 134.6)
- added DS5: 5161AS, HariLib:5161AS, F.Cu at (177.8, 50.8)
- added DS6: 5161AS, HariLib:5161AS, F.Cu at (190.5, 50.8)
- added DS7: 5161AS, HariLib:5161AS, F.Cu at (203.2, 50.8)
- added DS8: 5161AS, HariLib:5161AS, F.Cu at (215.9, 50.8)
- added DS9: 5161AS, HariLib:5161AS, F.Cu at (127.0, 71.1)
- U1, U2, U3, U4, U5, U7, U8: value 5161AS -> 74HC595; footprint HariLib:5161AS -> Package_SO:SOIC-16_3.9x9.9mm_P1.27mm
- U6: moved to F.Cu
- moved RN8 199.7 mm to (226.1, 157.5), turned to 90 degrees
- moved RN7 195.0 mm to (213.4, 157.5), turned to 90 degrees
- moved RN6 185.5 mm to (200.7, 157.5), turned to 90 degrees
- moved RN5 180.8 mm to (188.0, 157.5), turned to 90 degrees
- moved RN4 168.5 mm to (175.3, 157.5), turned to 90 degrees
- moved RN3 164.0 mm to (162.6, 157.5), turned to 90 degrees
- moved U7 141.5 mm to (210.8, 165.1), turned to 90 degrees
- moved U8 138.0 mm to (223.5, 165.1), turned to 90 degrees
- moved U1 132.6 mm to (134.6, 165.1), turned to 90 degrees
- moved U6 120.8 mm to (197.5, 165.2), turned to 90 degrees
- moved U5 117.8 mm to (185.4, 165.1), turned to 90 degrees
- moved U2 110.9 mm to (147.3, 165.1), turned to 90 degrees
- moved U4 109.1 mm to (172.7, 165.1), turned to 90 degrees
- moved U3 105.5 mm to (160.0, 165.1), turned to 90 degrees
- moved R4 92.0 mm to (119.4, 127.0), turned to 90 degrees
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Connections:
- Q1 pad 2: Net-(Q1-Pad2) -> Net-(DS1-Pad3)
- Q2 pad 2: Net-(Q2-Pad2) -> Net-(DS10-Pad3)
- Q3 pad 2: Net-(Q3-Pad2) -> Net-(DS17-Pad3)
- Q4 pad 2: Net-(Q4-Pad2) -> Net-(DS25-Pad3)
- Q5 pad 2: Net-(Q5-Pad2) -> Net-(DS33-Pad3)
- R1 pad 2: Net-(J1-Pad4) -> Net-(J1-Pad5)
- R2 pad 2: Net-(J1-Pad2) -> Net-(J1-Pad4)
- R3 pad 2: Net-(J1-Pad5) -> Net-(J1-Pad3)
- R4 pad 2: Net-(J1-Pad3) -> Net-(J1-Pad2)
- RN1 pad 10: Net-(RN1-Pad10) -> Net-(DS1-Pad10)
- RN1 pad 11: Net-(RN1-Pad11) -> Net-(DS1-Pad9)
- RN1 pad 12: Net-(RN1-Pad12) -> Net-(DS1-Pad1)
- RN1 pad 13: Net-(RN1-Pad13) -> Net-(DS1-Pad2)
- RN1 pad 14: Net-(RN1-Pad14) -> Net-(DS1-Pad4)
- RN1 pad 15: Net-(RN1-Pad15) -> Net-(DS1-Pad6)
- RN1 pad 16: Net-(RN1-Pad16) -> Net-(DS1-Pad7)
- RN1 pad 9: Net-(RN1-Pad9) -> Net-(DS1-Pad5)
- RN2 pad 10: Net-(RN2-Pad10) -> Net-(DS10-Pad10)
- RN2 pad 11: Net-(RN2-Pad11) -> Net-(DS10-Pad9)
- RN2 pad 12: Net-(RN2-Pad12) -> Net-(DS10-Pad1)
- RN2 pad 13: Net-(RN2-Pad13) -> Net-(DS10-Pad2)
- RN2 pad 14: Net-(RN2-Pad14) -> Net-(DS10-Pad4)
- RN2 pad 15: Net-(RN2-Pad15) -> Net-(DS10-Pad6)
- RN2 pad 16: Net-(RN2-Pad16) -> Net-(DS10-Pad7)
- RN2 pad 9: Net-(RN2-Pad9) -> Net-(DS10-Pad5)
- U1 pad 1: Net-(RN1-Pad12) -> Net-(RN1-Pad2)
- U1 pad 10: Net-(RN1-Pad10) -> +5V
- U1 pad 2: Net-(RN1-Pad13) -> Net-(RN1-Pad3)
- U1 pad 3: Net-(Q3-Pad2) -> Net-(RN1-Pad4)
- U1 pad 4: Net-(RN1-Pad14) -> Net-(RN1-Pad5)
- U1 pad 5: Net-(RN1-Pad9) -> Net-(RN1-Pad6)
- U1 pad 6: Net-(RN1-Pad15) -> Net-(RN1-Pad7)
- U1 pad 7: Net-(RN1-Pad16) -> Net-(RN1-Pad8)
- U1 pad 8: Net-(Q3-Pad2) -> GND
- U1 pad 9: Net-(RN1-Pad11) -> Net-(U1-Pad9)
- U2 pad 1: Net-(RN1-Pad12) -> Net-(RN2-Pad2)
- U2 pad 10: Net-(RN1-Pad10) -> +5V
- U2 pad 2: Net-(RN1-Pad13) -> Net-(RN2-Pad3)
- U2 pad 3: Net-(Q1-Pad2) -> Net-(RN2-Pad4)
- U2 pad 4: Net-(RN1-Pad14) -> Net-(RN2-Pad5)
- U2 pad 5: Net-(RN1-Pad9) -> Net-(RN2-Pad6)
- U2 pad 6: Net-(RN1-Pad15) -> Net-(RN2-Pad7)
- U2 pad 7: Net-(RN1-Pad16) -> Net-(RN2-Pad8)
- U2 pad 8: Net-(Q1-Pad2) -> GND
- U2 pad 9: Net-(RN1-Pad11) -> Net-(U2-Pad9)
- U3 pad 1: Net-(RN1-Pad12) -> Net-(RN3-Pad2)
- U3 pad 10: Net-(RN1-Pad10) -> +5V
- U3 pad 2: Net-(RN1-Pad13) -> Net-(RN3-Pad3)
- U3 pad 3: Net-(Q4-Pad2) -> Net-(RN3-Pad4)
- U3 pad 4: Net-(RN1-Pad14) -> Net-(RN3-Pad5)
- U3 pad 5: Net-(RN1-Pad9) -> Net-(RN3-Pad6)
- U3 pad 6: Net-(RN1-Pad15) -> Net-(RN3-Pad7)
- U3 pad 7: Net-(RN1-Pad16) -> Net-(RN3-Pad8)
- U3 pad 8: Net-(Q4-Pad2) -> GND
- U3 pad 9: Net-(RN1-Pad11) -> Net-(U3-Pad9)
- U4 pad 1: Net-(RN1-Pad12) -> Net-(RN4-Pad2)
- U4 pad 10: Net-(RN1-Pad10) -> +5V
- U4 pad 2: Net-(RN1-Pad13) -> Net-(RN4-Pad3)
- U4 pad 3: Net-(Q2-Pad2) -> Net-(RN4-Pad4)
- U4 pad 4: Net-(RN1-Pad14) -> Net-(RN4-Pad5)
- U4 pad 5: Net-(RN1-Pad9) -> Net-(RN4-Pad6)
- U4 pad 6: Net-(RN1-Pad15) -> Net-(RN4-Pad7)
- U4 pad 7: Net-(RN1-Pad16) -> Net-(RN4-Pad8)
- U4 pad 8: Net-(Q2-Pad2) -> GND
- U4 pad 9: Net-(RN1-Pad11) -> Net-(U4-Pad9)
- U5 pad 1: Net-(RN1-Pad12) -> Net-(RN5-Pad2)
- U5 pad 10: Net-(RN1-Pad10) -> +5V
- U5 pad 2: Net-(RN1-Pad13) -> Net-(RN5-Pad3)
- U5 pad 3: Net-(Q5-Pad2) -> Net-(RN5-Pad4)
- U5 pad 4: Net-(RN1-Pad14) -> Net-(RN5-Pad5)
- U5 pad 5: Net-(RN1-Pad9) -> Net-(RN5-Pad6)
- U5 pad 6: Net-(RN1-Pad15) -> Net-(RN5-Pad7)
- U5 pad 7: Net-(RN1-Pad16) -> Net-(RN5-Pad8)
- U5 pad 8: Net-(Q5-Pad2) -> GND
- U5 pad 9: Net-(RN1-Pad11) -> Net-(U5-Pad9)
- U6 pad 1: Net-(RN1-Pad2) -> Net-(RN6-Pad2)
- U6 pad 14: Net-(J2-Pad1) -> Net-(U5-Pad9)
- U6 pad 15: Net-(RN1-Pad1) -> Net-(RN6-Pad1)
- U6 pad 2: Net-(RN1-Pad3) -> Net-(RN6-Pad3)
- U6 pad 3: Net-(RN1-Pad4) -> Net-(RN6-Pad4)
- U6 pad 4: Net-(RN1-Pad5) -> Net-(RN6-Pad5)
- U6 pad 5: Net-(RN1-Pad6) -> Net-(RN6-Pad6)
- U6 pad 6: Net-(RN1-Pad7) -> Net-(RN6-Pad7)
- U6 pad 7: Net-(RN1-Pad8) -> Net-(RN6-Pad8)
- U6 pad 9: Net-(U12-Pad14) -> Net-(U6-Pad9)
- U7 pad 1: Net-(RN2-Pad12) -> Net-(RN7-Pad2)
- U7 pad 10: Net-(RN2-Pad10) -> +5V
- U7 pad 2: Net-(RN2-Pad13) -> Net-(RN7-Pad3)
- U7 pad 3: Net-(Q3-Pad2) -> Net-(RN7-Pad4)
- U7 pad 4: Net-(RN2-Pad14) -> Net-(RN7-Pad5)
- U7 pad 5: Net-(RN2-Pad9) -> Net-(RN7-Pad6)
- U7 pad 6: Net-(RN2-Pad15) -> Net-(RN7-Pad7)
- U7 pad 7: Net-(RN2-Pad16) -> Net-(RN7-Pad8)
- U7 pad 8: Net-(Q3-Pad2) -> GND
- U7 pad 9: Net-(RN2-Pad11) -> Net-(U7-Pad9)
- U8 pad 1: Net-(RN2-Pad12) -> Net-(RN8-Pad2)
- U8 pad 10: Net-(RN2-Pad10) -> +5V
- U8 pad 2: Net-(RN2-Pad13) -> Net-(RN8-Pad3)
- U8 pad 3: Net-(Q1-Pad2) -> Net-(RN8-Pad4)
- U8 pad 4: Net-(RN2-Pad14) -> Net-(RN8-Pad5)
- U8 pad 5: Net-(RN2-Pad9) -> Net-(RN8-Pad6)
- U8 pad 6: Net-(RN2-Pad15) -> Net-(RN8-Pad7)
- U8 pad 7: Net-(RN2-Pad16) -> Net-(RN8-Pad8)
- U8 pad 8: Net-(Q1-Pad2) -> GND
- U8 pad 9: Net-(RN2-Pad11) -> (no net)
Routing:
- net Net-(RN1-Pad12): track 53.6 -> 0.00 mm
- net Net-(Q5-Pad2): track 53.1 -> 0.00 mm, vias 2 -> 0
- net Net-(RN1-Pad10): track 52.9 -> 0.00 mm
- net Net-(RN1-Pad13): track 50.8 -> 0.00 mm, vias 2 -> 0
- net Net-(RN1-Pad11): track 47.5 -> 0.00 mm, vias 2 -> 0
- net Net-(RN1-Pad9): track 45.6 -> 0.00 mm
- net Net-(RN1-Pad15): track 41.9 -> 0.00 mm, vias 2 -> 0
- net Net-(J2-Pad3): track 41.7 -> 0.00 mm, vias 2 -> 0
- net Net-(RN1-Pad16): track 41.0 -> 0.00 mm
- net Net-(J2-Pad2): track 38.9 -> 0.00 mm, vias 2 -> 0
- net +5V: track 32.0 -> 0.00 mm
- net Net-(RN2-Pad12): track 31.8 -> 0.00 mm
- net Net-(RN2-Pad13): track 29.8 -> 0.00 mm, vias 2 -> 0
- net Net-(RN2-Pad10): track 29.7 -> 0.00 mm
- net Net-(RN2-Pad11): track 26.6 -> 0.00 mm, vias 2 -> 0
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- removed copper zone on B.Cu, net GND

Commit message: About to try FreeRouting
Parts:
- moved DS37 12.7 mm to (167.6, 127.0)
- moved U6 12.7 mm to (187.3, 157.5)
- moved U1 12.7 mm to (124.5, 157.5)
- moved RN2 12.7 mm to (139.7, 149.9)
- moved RN7 12.7 mm to (203.2, 149.9)
- moved DS33 12.7 mm to (116.8, 127.0)
- moved DS34 12.7 mm to (129.5, 127.0)
- moved DS35 12.7 mm to (142.2, 127.0)
- moved DS36 12.7 mm to (154.9, 127.0)
- moved DS38 12.7 mm to (180.3, 127.0)
- moved DS39 12.7 mm to (193.0, 127.0)
- moved DS40 12.7 mm to (205.7, 127.0)
- moved U2 12.7 mm to (137.2, 157.5)
- moved U3 12.7 mm to (149.9, 157.5)
- moved U4 12.7 mm to (162.6, 157.5)
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Routing:
- net Net-(DS1-Pad3): track 0.00 -> 236.5 mm
- net Net-(DS10-Pad3): track 0.00 -> 231.1 mm
- net Net-(DS25-Pad3): track 0.00 -> 224.7 mm
- net Net-(DS33-Pad3): track 0.00 -> 223.4 mm
- net Net-(DS17-Pad3): track 0.00 -> 207.6 mm
- net Net-(DS16-Pad10): track 0.00 -> 113.1 mm, vias 0 -> 2
- net Net-(DS15-Pad10): track 0.00 -> 113.1 mm, vias 0 -> 1
- net Net-(DS16-Pad7): track 0.00 -> 102.2 mm
- net Net-(DS16-Pad6): track 0.00 -> 101.5 mm
- net Net-(DS16-Pad1): track 0.00 -> 93.0 mm
- net Net-(DS16-Pad2): track 0.00 -> 90.1 mm
- net Net-(DS16-Pad4): track 0.00 -> 86.0 mm, vias 0 -> 2
- net Net-(DS15-Pad5): track 0.00 -> 85.4 mm
- net Net-(DS16-Pad5): track 0.00 -> 85.4 mm
- net Net-(DS16-Pad9): track 0.00 -> 80.4 mm
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
Commit message: FreeRouting appears to be stuck routing so did it by hand afterall.
Parts:
- added J3: 22-23-2021, Connector_PinHeader_2.54mm:PinHeader_1x02_P2.54mm_Vertical, F.Cu at (106.7, 144.8)
- J1: footprint Connector_PinHeader_2.00mm:PinHeader_1x05_P2.00mm_Vertical -> Connector_PinHeader_2.54mm:PinHeader_1x05_P2.54mm_Vertical
- J2: footprint Connector_PinHeader_2.00mm:PinHeader_1x03_P2.00mm_Vertical -> Connector_PinHeader_2.54mm:PinHeader_1x03_P2.54mm_Vertical
- moved J2 7.70 mm to (106.7, 154.9)
Routing:
- net +5V: track 0.00 -> 169.0 mm, vias 0 -> 16
- net Net-(J2-Pad3): track 0.00 -> 140.8 mm, vias 0 -> 9
- net Net-(J2-Pad2): track 0.00 -> 124.0 mm, vias 0 -> 8
- net Net-(DS10-Pad7): track 0.00 -> 103.9 mm
- net Net-(DS14-Pad7): track 0.00 -> 102.0 mm
- net Net-(DS1-Pad7): track 0.00 -> 102.0 mm
- net Net-(DS15-Pad7): track 0.00 -> 102.0 mm
- net Net-(DS15-Pad6): track 0.00 -> 101.5 mm
- net Net-(DS13-Pad6): track 0.00 -> 101.5 mm
- net Net-(DS10-Pad6): track 0.00 -> 101.5 mm
- net Net-(DS11-Pad6): track 0.00 -> 101.5 mm
- net Net-(DS1-Pad6): track 0.00 -> 101.5 mm
- net Net-(DS14-Pad6): track 0.00 -> 101.5 mm
- net Net-(DS12-Pad6): track 0.00 -> 101.5 mm
- net Net-(DS12-Pad7): track 0.00 -> 101.1 mm
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- added copper zone on B.Cu, net GND
Other:
- board text added: "+5V"
- board text added: "1"
- board text added: "CLK"
- board text added: "GND"
- board text added: "LATCH"
- board text added: "SER"
